File: EAGLE/schema-projet-elec.brd (EAGLE design)
At the start: 100 x 80 mm, 25 parts

Commit message: Change brd ans sch
Parts:
- removed D1: RED, SparkFun-LED:LED-0603
- removed D2: GREEN, SparkFun-LED:LED-0603
- added GREEN, RED: (no value), SparkFun-LED:LED_5MM
- moved R4 17.3 mm to (88.2, 76.2), turned to 0 degrees
- moved R11 16.5 mm to (69.8, 51.8)
- moved R19 16.2 mm to (31.6, 53.2)
- moved R13 15.1 mm to (31.6, 44.8)
- moved R8 14.8 mm to (74.5, 39.6)
- moved R15 13.8 mm to (31.3, 36.8)
- moved R7 13.7 mm to (70.4, 35.6)
- moved R17 13.3 mm to (31.8, 29.2)
- moved R5 13.0 mm to (70.2, 27.6)
- moved R12 12.9 mm to (27.7, 48.8)
- moved R9 12.4 mm to (70.7, 43.6)
- moved R10 12.3 mm to (74.8, 47.6), turned to 0 degrees
- moved R14 11.2 mm to (27.4, 40.8)
- moved R6 9.75 mm to (74.3, 31.6), flipped to the top, turned to 0 degrees
- moved R16 9.75 mm to (27.2, 32.8)
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Connections:
- net N$2: now also RED.A; no longer D1.A
- net N$4: now also GREEN.A; no longer D2.A
- net N$5: now also GREEN.K, RED.K; no longer D1.C, D2.C
Routing:
- net N$42: track 26.8 -> 115.3 mm
- net N$41: track 74.2 -> 138.2 mm
- net N$31: track 55.9 -> 105.8 mm
- net N$5: track 19.6 -> 65.7 mm
- net N$4: track 4.19 -> 32.0 mm
- net N$13: track 44.0 -> 69.6 mm
- net N$44: track 27.5 -> 48.8 mm
- net N$19: track 25.8 -> 8.88 mm
- net N$22: track 23.7 -> 7.85 mm
- net N$39: track 22.7 -> 7.40 mm
- net N$7: track 32.3 -> 47.6 mm
- net N$26: track 32.5 -> 18.8 mm
- net N$18: track 25.8 -> 12.3 mm
- net N$32: track 21.7 -> 8.61 mm
- net N$20: track 24.8 -> 12.4 mm
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- added copper zone on layer 16, net GND
Other:
- board text added: "Groupe 3 Samuel Lambert Julien Pollart Martin Hayot Gaetan Leplae Basil Huwart"

Commit message: Add files via upload
Parts:
- removed GREEN, RED: (no value), SparkFun-LED:LED_5MM
- added LED1, LED2: (no value), led:LED5MM
Connections:
- net N$2: now also LED1.A; no longer RED.A
- net N$4: now also LED2.A; no longer GREEN.A
- net N$5: now also LED1.K, LED2.K; no longer GREEN.K, RED.K
Routing:
- net N$4: track 32.0 -> 9.42 mm
- net N$2: track 6.27 -> 8.36 mm
- net N$5: track 65.7 -> 64.0 mm
